File: hardware/rs485if/rs485if.sch (EAGLE design)
At the start: 78 parts, among them IC1 BSP75, IC2 PCA82C250SMD, IC4 78L05SMD, IC5 MAX481CSA, Q1 3M6864, T1 MKDSO_2.5/3_R, T2 MKDSO_2.5/3_R, T3 MKDSO_2.5/3_L, T4 MKDSO_2.5/3_L

Commit message: part value actualization
Parts:
- C14: value (none) -> 10n
- D14, D7: value (none) -> 1N4148
- D6: value 7V5 -> 6V2
- Q1: value 3M6864 -> 18M432
- R4: value (none) -> 100k
- R5: value (none) -> 4k7
- U$3: value (none) -> Atmega1284
Other:
- note added: "Housing: Phoenix Contact BC 17,8"
Changed lines of the file:
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@@
 <part name="C2" library="rcl" deviceset="CPOL-EU" device="A/3216-18W" value="10µ/10V"/>
 <part name="GND1" library="supply1" deviceset="GND" device=""/>
-<part name="Q1" library="crystal" deviceset="CRYSTAL" device="SM49" value="3M6864"/>
+<part name="Q1" library="crystal" deviceset="CRYSTAL" device="SM49" value="18M432"/>
 <part name="GND6" library="supply1" deviceset="GND" device=""/>
 <part name="C4" library="resistor" deviceset="C-EU" device="C0603" value="16p"/>
@@
 <part name="GND10" library="supply1" deviceset="GND" device=""/>
 <part name="GND5" library="supply1" deviceset="GND" device=""/>
-<part name="D7" library="diode" deviceset="DIODE-" device="SOD80C"/>
-<part name="R5" library="resistor" deviceset="R-EU_" device="R0603"/>
-<part name="C14" library="resistor" deviceset="C-EU" device="C0603"/>
+<part name="D7" library="diode" deviceset="DIODE-" device="SOD80C" value="1N4148"/>
+<part name="R5" library="resistor" deviceset="R-EU_" device="R0603" value="4k7"/>
+<part name="C14" library="resistor" deviceset="C-EU" device="C0603" value="10n"/>
 <part name="GND16" library="supply1" deviceset="GND" device=""/>
 <part name="GND17" library="supply1" deviceset="GND" device=""/>
@@
 <part name="R3" library="resistor" deviceset="R-EU_" device="R0603" value="10k"/>
 <part name="GND20" library="supply1" deviceset="GND" device=""/>
-<part name="U$3" library="mylib" deviceset="ATMEGA644" device=""/>
+<part name="U$3" library="mylib" deviceset="ATMEGA644" device="" value="Atmega1284"/>
 <part name="IC1" library="mylib" deviceset="BSP75" device=""/>
 <part name="GND21" library="supply1" deviceset="GND" device=""/>
@@
 <part name="R19" library="resistor" deviceset="R-EU_" device="R0603" value="2k2"/>
 <part name="R20" library="resistor" deviceset="R-EU_" device="R0603" value="2k2"/>
-<part name="D6" library="diode" deviceset="ZENER-DIODE" device="SOD80C" value="7V5"/>
+<part name="D6" library="diode" deviceset="ZENER-DIODE" device="SOD80C" value="6V2"/>
 <part name="JP3" library="pinhead" deviceset="PINHD-1X2" device="" value="RESET"/>
 <part name="GND31" library="supply1" deviceset="GND" device=""/>
@@
 <part name="GND33" library="supply1" deviceset="GND" device=""/>
 <part name="SJ1" library="jumper" deviceset="SJ" device=""/>
-<part name="R4" library="resistor" deviceset="R-EU_" device="R0603"/>
-<part name="D14" library="diode" deviceset="DIODE-" device="SOD80C"/>
+<part name="R4" library="resistor" deviceset="R-EU_" device="R0603" value="100k"/>
+<part name="D14" library="diode" deviceset="DIODE-" device="SOD80C" value="1N4148"/>
 <part name="P+3" library="supply1" deviceset="VCC" device=""/>
 <part name="C21" library="resistor" deviceset="C-EU" device="C0603" value="100n"/>
@@
 <plain>
 <text x="71.12" y="20.32" size="1.778" layer="97" rot="R180">Power fail interrupt</text>
+<text x="238.76" y="134.62" size="2.54" layer="97">Housing: Phoenix Contact BC 17,8</text>
 </plain>
 <instances>
