File: hardware/pwm4/pwm4.brd (EAGLE design)
At the start: 102 x 39 mm, 79 parts, among them IC1 BSP75, IC2 PCA82C250SMD, IC3 BSP75, IC4 78L05SMD, IC6 BSP75, IC7 BSP75, Q1 18M432

Commit message: changed crystal frequency
Parts:
- Q1: value 18M432 -> 14M7456
Changed lines of the file:
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@@
 <element name="C1" library="resistor" package="C0603" value="100n" x="84.5312" y="27.1272" rot="R90"/>
 <element name="C2" library="rcl" package="A/3216-18W" value="10µ/10V" x="86.5632" y="26.162" rot="MR0"/>
-<element name="Q1" library="crystal" package="SM49" value="18M432" x="96.5582" y="13.739" rot="R90">
+<element name="Q1" library="crystal" package="SM49" value="14M7456" x="96.5582" y="13.739" rot="R90">
 <attribute name="OC_NEWARK" value="unknown" x="143.5482" y="49.299" size="1.778" layer="27" rot="R90" display="off"/>
 <attribute name="MPN" value="" x="143.5482" y="49.299" size="1.778" layer="27" rot="R90" display="off"/>

Commit message: optocoupler input and output resistor change
Parts:
- C22, C26, C6, C8: value 2n2 -> n.b.
- R1, R2, R3, R6: value 680 -> 1k2
- R10, R11, R7, R9: value 1k -> 2k2
- renumbered U$10 to BUS, U$5 to PWM0, U$6 to PWM1, U$7 to PWM2, U$8 to PWM3, U$9 to 24V
Connections:
- net N$33 renamed PWM1
- net N$34 renamed PWM2
- net N$35 renamed PWM0
- net N$5 renamed MOSI
- net N$6 renamed MISO
- net N$7 renamed SCK
- net N$8 renamed PWM3
Changed lines of the file:
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@@
 <element name="D15" library="diode" package="SMB" value="SS24" x="34.036" y="15.24" rot="R270"/>
 <element name="U$4" library="mylib" package="SOIC16" value="TCMT4100" x="63.1952" y="9.906" rot="R90"/>
-<element name="R1" library="resistor" package="R0603" value="680" x="69.9008" y="5.2832"/>
-<element name="R2" library="resistor" package="R0603" value="680" x="70.866" y="8.7376" rot="R90"/>
-<element name="R3" library="resistor" package="R0603" value="680" x="70.358" y="12.5476" rot="R90"/>
-<element name="R6" library="resistor" package="R0603" value="680" x="70.7136" y="15.1384"/>
-<element name="R7" library="resistor" package="R0603" value="1k" x="6.2992" y="23.7744" rot="R180"/>
-<element name="R9" library="resistor" package="R0603" value="1k" x="21.2852" y="23.7744" rot="R180"/>
-<element name="R10" library="resistor" package="R0603" value="1k" x="37.0332" y="23.7236" rot="R180"/>
-<element name="R11" library="resistor" package="R0603" value="1k" x="51.3588" y="23.7744" rot="R180"/>
-<element name="U$5" library="mylib" package="TBG-3.5-PW-2P" value="TBG-3.5-PW-2P" x="12.446" y="35.1028" rot="MR270"/>
-<element name="U$6" library="mylib" package="TBG-3.5-PW-2P" value="TBG-3.5-PW-2P" x="27.5336" y="35.1028" rot="MR270"/>
-<element name="U$7" library="mylib" package="TBG-3.5-PW-2P" value="TBG-3.5-PW-2P" x="42.5196" y="35.1028" rot="MR270"/>
-<element name="U$8" library="mylib" package="TBG-3.5-PW-2P" value="TBG-3.5-PW-2P" x="57.5564" y="35.1028" rot="MR270"/>
-<element name="U$9" library="mylib" package="TBG-3.5-PW-2P" value="TBG-3.5-PW-2P" x="9.7028" y="5.08" rot="MR0"/>
-<element name="U$10" library="mylib" package="TBG-3.5-PW-4P" value="TBG-3.5-PW-4P" x="85.4964" y="32.9184" rot="MR180"/>
+<element name="R1" library="resistor" package="R0603" value="1k2" x="69.9008" y="5.2832"/>
+<element name="R2" library="resistor" package="R0603" value="1k2" x="70.866" y="8.7376" rot="R90"/>
+<element name="R3" library="resistor" package="R0603" value="1k2" x="70.358" y="12.5476" rot="R90"/>
+<element name="R6" library="resistor" package="R0603" value="1k2" x="70.7136" y="15.1384"/>
+<element name="R7" library="resistor" package="R0603" value="2k2" x="6.2992" y="23.7744" rot="R180"/>
+<element name="R9" library="resistor" package="R0603" value="2k2" x="21.2852" y="23.7744" rot="R180"/>
+<element name="R10" library="resistor" package="R0603" value="2k2" x="37.0332" y="23.7236" rot="R180"/>
+<element name="R11" library="resistor" package="R0603" value="2k2" x="51.3588" y="23.7744" rot="R180"/>
+<element name="PWM0" library="mylib" package="TBG-3.5-PW-2P" value="TBG-3.5-PW-2P" x="12.446" y="35.1028" rot="MR270"/>
+<element name="PWM1" library="mylib" package="TBG-3.5-PW-2P" value="TBG-3.5-PW-2P" x="27.5336" y="35.1028" rot="MR270"/>
+<element name="PWM2" library="mylib" package="TBG-3.5-PW-2P" value="TBG-3.5-PW-2P" x="42.5196" y="35.1028" rot="MR270"/>
+<element name="PWM3" library="mylib" package="TBG-3.5-PW-2P" value="TBG-3.5-PW-2P" x="57.5564" y="35.1028" rot="MR270"/>
+<element name="24V" library="mylib" package="TBG-3.5-PW-2P" value="TBG-3.5-PW-2P" x="9.7028" y="5.08" rot="MR0"/>
+<element name="BUS" library="mylib" package="TBG-3.5-PW-4P" value="TBG-3.5-PW-4P" x="85.4964" y="32.9184" rot="MR180"/>
 <element name="D11" library="diode" package="SMC" value="SMCJ30A" x="16.8148" y="5.08" rot="R180"/>
 <element name="U$2" library="mega32U4" package="TQFP44" value="ATMEGA32U4-AU" x="84.0232" y="14.1732" rot="R90"/>
-<element name="C6" library="resistor" package="C025-040X050" value="2n2" x="12.8524" y="24.2824" rot="R180"/>
+<element name="C6" library="resistor" package="C025-040X050" value="n.b." x="12.8524" y="24.2824" rot="R180"/>
 <element name="C7" library="resistor" package="C025-040X050" value="2n2" x="27.6352" y="28.194" rot="R180"/>
-<element name="C8" library="resistor" package="C025-040X050" value="2n2" x="27.6352" y="24.2316" rot="R180"/>
+<element name="C8" library="resistor" package="C025-040X050" value="n.b." x="27.6352" y="24.2316" rot="R180"/>
 <element name="C17" library="resistor" package="C025-040X050" value="2n2" x="43.0784" y="28.1432" rot="R180"/>
-<element name="C22" library="resistor" package="C025-040X050" value="2n2" x="43.0784" y="24.1808" rot="R180"/>
+<element name="C22" library="resistor" package="C025-040X050" value="n.b." x="43.0784" y="24.1808" rot="R180"/>
 <element name="C24" library="resistor" package="C025-040X050" value="2n2" x="57.404" y="28.194" rot="R180"/>
-<element name="C26" library="resistor" package="C025-040X050" value="2n2" x="57.404" y="24.1808" rot="R180"/>
+<element name="C26" library="resistor" package="C025-040X050" value="n.b." x="57.404" y="24.1808" rot="R180"/>
 <element name="C27" library="resistor" package="C025-040X050" value="2n2" x="24.8412" y="3.9624" rot="R90"/>
 <element name="C28" library="resistor" package="C025-040X050" value="2n2" x="29.0576" y="3.9624" rot="R90"/>
@@
 <contactref element="U$4" pad="6"/>
 <contactref element="U$4" pad="8"/>
-<contactref element="U$10" pad="P$2"/>
+<contactref element="BUS" pad="P$2"/>
 <contactref element="U$2" pad="15"/>
 <contactref element="U$2" pad="23"/>
@@
 <wire x1="82.8684" y1="27.9772" x2="82.8548" y2="27.9908" width="0.4064" layer="1"/>
 </signal>
-<signal name="N$5">
+<signal name="MOSI">
 <contactref element="U$1" pad="PAD3"/>
 <contactref element="U$2" pad="10"/>
@@
 <wire x1="90.2997" y1="4.4196" x2="90.3505" y2="4.3688" width="0.254" layer="1"/>
 </signal>
-<signal name="N$6">
+<signal name="MISO">
 <contactref element="U$1" pad="PAD2"/>
 <contactref element="U$2" pad="11"/>
@@
 <wire x1="88.8852" y1="7.5112" x2="88.8852" y2="5.8341" width="0.254" layer="1"/>
 </signal>
-<signal name="N$7">
+<signal name="SCK">
 <contactref element="U$1" pad="PAD6"/>
 <contactref element="U$2" pad="9"/>
@@
 <contactref element="D1" pad="1"/>
 <contactref element="L4" pad="4"/>
-<contactref element="U$10" pad="P$3"/>
+<contactref element="BUS" pad="P$3"/>
 <wire x1="92.4964" y1="32.9184" x2="91.5944" y2="32.0164" width="0.4064" layer="16"/>
 <wire x1="91.5944" y1="32.0164" x2="91.5944" y2="28.5146" width="0.4064" layer="16"/>
@@
 <contactref element="D2" pad="1"/>
 <contactref element="L4" pad="3"/>
-<contactref element="U$10" pad="P$4"/>
+<contactref element="BUS" pad="P$4"/>
 <wire x1="95.9964" y1="32.9184" x2="95.8108" y2="32.7328" width="0.4064" layer="16"/>
 <wire x1="95.8108" y1="32.7328" x2="95.8108" y2="28.667" width="0.4064" layer="16"/>
@@
 <wire x1="81.026" y1="33.8328" x2="81.3036" y2="33.8328" width="0.254" layer="1"/>
 </signal>
-<signal name="N$8">
+<signal name="PWM3">
 <contactref element="R6" pad="2"/>
 <contactref element="U$2" pad="29"/>
@@
 <wire x1="83.2232" y1="21.2216" x2="83.2232" y2="19.9732" width="0.254" layer="1"/>
 </signal>
-<signal name="N$33">
+<signal name="PWM1">
 <contactref element="R2" pad="2"/>
 <contactref element="U$2" pad="32"/>
@@
 <wire x1="80.8232" y1="21.336" x2="80.8232" y2="19.9732" width="0.254" layer="1"/>
 </signal>
-<signal name="N$34">
+<signal name="PWM2">
 <contactref element="R3" pad="2"/>
 <contactref element="U$2" pad="30"/>
@@
 <wire x1="71.5264" y1="33.352" x2="71.5264" y2="27.4692" width="0.254" layer="1"/>
 </signal>
-<signal name="N$35">
+<signal name="PWM0">
 <contactref element="U$2" pad="12"/>
 <contactref element="R1" pad="2"/>
@@
 <contactref element="C3" pad="2"/>
 <contactref element="D5" pad="C"/>
-<contactref element="U$5" pad="P$2"/>
+<contactref element="PWM0" pad="P$2"/>
 <contactref element="C6" pad="2"/>
 <wire x1="6.35" y1="36.4152" x2="7.6336" y2="36.4152" width="1.27" layer="1"/>
@@
 <contactref element="IC3" pad="2"/>
 <contactref element="D8" pad="C"/>
-<contactref element="U$6" pad="P$2"/>
+<contactref element="PWM1" pad="P$2"/>
 <contactref element="C7" pad="2"/>
 <contactref element="C8" pad="2"/>
@@
 <contactref element="IC6" pad="2"/>
 <contactref element="D9" pad="C"/>
-<contactref element="U$7" pad="P$2"/>
+<contactref element="PWM2" pad="P$2"/>
 <contactref element="C17" pad="2"/>
 <contactref element="C22" pad="2"/>
@@
 <contactref element="IC7" pad="2"/>
 <contactref element="D10" pad="C"/>
-<contactref element="U$8" pad="P$2"/>
+<contactref element="PWM3" pad="P$2"/>
 <contactref element="C24" pad="2"/>
 <contactref element="C26" pad="2"/>
@@
 <contactref element="D15" pad="C"/>
 <contactref element="D13" pad="C"/>
-<contactref element="U$5" pad="P$1"/>
-<contactref element="U$6" pad="P$1"/>
-<contactref element="U$7" pad="P$1"/>
-<contactref element="U$8" pad="P$1"/>
+<contactref element="PWM0" pad="P$1"/>
+<contactref element="PWM1" pad="P$1"/>
+<contactref element="PWM2" pad="P$1"/>
+<contactref element="PWM3" pad="P$1"/>
 <contactref element="D11" pad="C"/>
 <contactref element="C27" pad="2"/>
@@
 <contactref element="R9" pad="1"/>
 <contactref element="R7" pad="1"/>
-<contactref element="U$9" pad="P$1"/>
+<contactref element="24V" pad="P$1"/>
 <contactref element="D11" pad="A"/>
 <contactref element="C7" pad="1"/>
@@
 <signal name="N$21">
 <contactref element="F1" pad="2A"/>
-<contactref element="U$9" pad="P$2"/>
+<contactref element="24V" pad="P$2"/>
 <wire x1="6.2028" y1="5.08" x2="6.2028" y2="14.0208" width="1.6764" layer="1"/>
 <wire x1="6.2028" y1="14.0208" x2="9.652" y2="14.0208" width="1.6764" layer="1"/>
@@
 <signal name="N$20">
 <contactref element="L1" pad="2"/>
-<contactref element="U$10" pad="P$1"/>
+<contactref element="BUS" pad="P$1"/>
 <contactref element="D4" pad="C"/>
 <wire x1="81.3504" y1="36.6776" x2="81.8584" y2="36.1696" width="0.4064" layer="1"/>
