File: hardware/smartmeterif/smartmeterif.brd (EAGLE design)
At the start: 84.3 x 51 mm, 47 parts, among them IC1 AT90USB647-AU, IC2 PCA82C250SMD, IC3 USBLC6, Q1 8M, Q2 BSS315, Q3 BC846BSMD, X1 PN87520-S

Commit message: smartmeterif hardware: value changes
Parts:
- R10, R7: value 1k -> 1k n.b.
- R9: value 10k -> 2k2
Changed lines of the file:
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@@
 <?xml version="1.0" encoding="utf-8"?>
 <!DOCTYPE eagle SYSTEM "eagle.dtd">
-<eagle version="6.5.0">
+<eagle version="7.1.0">
 <drawing>
 <settings>
@@
 <pass name="Default">
 <param name="RoutingGrid" value="50mil"/>
+<param name="AutoGrid" value="1"/>
+<param name="Efforts" value="0"/>
+<param name="TopRouterVariant" value="1"/>
 <param name="tpViaShape" value="round"/>
 <param name="PrefDir.1" value="|"/>
@@
 <element name="C17" library="resistor" package="C0603" value="100n" x="55.4228" y="39.1668" rot="MR180"/>
 <element name="L6" library="rcl" package="L1812" value="6µ8/0A6" x="55.4482" y="36.322" rot="R180"/>
-<element name="R7" library="rcl" package="R0603" value="1k" x="35.0012" y="26.6192" rot="MR180"/>
+<element name="R7" library="rcl" package="R0603" value="1k n.b." x="35.0012" y="26.6192" rot="MR180"/>
 <element name="U$3" library="mylib" package="PHOENIX_MKDSO_2.5/3_L" value="MKDSO_2.5/3_L" x="78.0542" y="13.7668"/>
 <element name="U$4" library="mylib" package="PHOENIX_MKDSO_2.5/3_L" value="MKDSO_2.5/3_L" x="68.0212" y="31.2674"/>
 <element name="JP1" library="pinhead" package="1X02" value="LED" x="26.924" y="45.9486"/>
-<element name="R9" library="resistor" package="R0603" value="10k" x="27.178" y="40.64" rot="R270"/>
+<element name="R9" library="resistor" package="R0603" value="2k2" x="27.178" y="40.64" rot="R270"/>
 <element name="C18" library="rcl" package="SMC_A" value="4µ7/10V" x="47.7266" y="47.0916" rot="R90"/>
-<element name="R10" library="rcl" package="R0603" value="1k" x="36.1188" y="11.5824" rot="MR270"/>
+<element name="R10" library="rcl" package="R0603" value="1k n.b." x="36.1188" y="11.5824" rot="MR270"/>
 </elements>
 <signals>
