File: hardware/smartmeterif/smartmeterif.sch (EAGLE design)
At the start: 46 parts, among them IC1 AT90USB647-AU, IC2 PCA82C250SMD, IC3 USBLC6, Q1 8M, Q2 BSS315, Q3 BC846BSMD, X1 PN87520-S

Commit message: smartmeterif hardware: value changes
Parts:
- R10, R7: value 1k -> 1k n.b.
- R9: value 10k -> 2k2
Changed lines of the file:
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@@
 <?xml version="1.0" encoding="utf-8"?>
 <!DOCTYPE eagle SYSTEM "eagle.dtd">
-<eagle version="6.5.0">
+<eagle version="7.1.0">
 <drawing>
 <settings>
@@
 <part name="GND25" library="supply1" deviceset="GND" device=""/>
 <part name="L6" library="rcl" deviceset="L-EU" device="L1812" value="6µ8/0A6"/>
-<part name="R7" library="rcl" deviceset="R-EU_" device="R0603" value="1k"/>
+<part name="R7" library="rcl" deviceset="R-EU_" device="R0603" value="1k n.b."/>
 <part name="GND26" library="supply1" deviceset="GND" device=""/>
 <part name="U$3" library="mylib" deviceset="MKDSO_2.5/3_L" device=""/>
@@
 <part name="GND28" library="supply1" deviceset="GND" device=""/>
 <part name="JP1" library="pinhead" deviceset="PINHD-1X2" device="" value="LED"/>
-<part name="R9" library="resistor" deviceset="R-EU_" device="R0603" value="10k"/>
+<part name="R9" library="resistor" deviceset="R-EU_" device="R0603" value="2k2"/>
 <part name="GND3" library="supply1" deviceset="GND" device=""/>
 <part name="C18" library="rcl" deviceset="CPOL-EU" device="SMCA" value="4µ7/10V"/>
 <part name="GND29" library="supply1" deviceset="GND" device=""/>
-<part name="R10" library="rcl" deviceset="R-EU_" device="R0603" value="1k"/>
+<part name="R10" library="rcl" deviceset="R-EU_" device="R0603" value="1k n.b."/>
 <part name="GND30" library="supply1" deviceset="GND" device=""/>
 </parts>
