File: hardware/do8/do8.kicad_sch (KiCad schematic)
At the start: 46 parts, among them J3 PHOENIX_MKDSO_2.5_3_L, J4 PHOENIX_MKDSO_2.5_3_L, J5 PHOENIX_MKDSO_2.5_3_R, J6 PHOENIX_MKDSO_2.5_3_R, Q1 BSP75N, Q2 BSP75N, Q3 BSP75N, Q4 BSP75N, Q5 BSP75N, Q6 BSP75N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

Commit message: Ordered PCB
Parts:
- U1: footprint mylib:phoenix-bc178-reduced-1 -> mylib:phoenix-bc178-reduced-3
Connections:
- net PB7: now reaches U2.12 (PB7)
Changed lines of the file:
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@@
 		)
 	)
+	(label "PB7"
+		(at 81.28 68.58 0)
+		(effects
+			(font
+				(size 1.27 1.27)
+			)
+			(justify left bottom)
+		)
+	)
 	(label "DO0"
 		(at 261.62 95.25 0)
@@
 			)
 		)
-		(property "Footprint" "mylib:phoenix-bc178-reduced-1"
+		(property "Footprint" "mylib:phoenix-bc178-reduced-3"
 			(at 45.72 16.51 0)
 			(hide yes)
@@
 		(in_pos_files yes)
 		(dnp no)
-		(fields_autoplaced yes)
 		(property "Reference" "J4"
-			(at 284.48 153.6699 0)
+			(at 280.924 146.05 0)
 			(show_name no)
 			(do_not_autoplace no)
@@
 		)
 		(property "Value" "PHOENIX_MKDSO_2.5_3_L"
-			(at 284.48 156.2099 0)
+			(at 259.08 148.082 0)
 			(show_name no)
 			(do_not_autoplace no)
@@
 		(in_pos_files yes)
 		(dnp no)
-		(fields_autoplaced yes)
 		(property "Reference" "J3"
-			(at 284.48 119.3799 0)
+			(at 280.416 111.506 0)
 			(show_name no)
 			(do_not_autoplace no)
@@
 		)
 		(property "Value" "PHOENIX_MKDSO_2.5_3_L"
-			(at 284.48 121.9199 0)
+			(at 259.08 113.538 0)
 			(show_name no)
 			(do_not_autoplace no)
@@
 		(in_pos_files yes)
 		(dnp no)
-		(fields_autoplaced yes)
 		(property "Reference" "J5"
-			(at 284.48 72.3899 0)
+			(at 280.416 64.262 0)
 			(show_name no)
 			(do_not_autoplace no)
@@
 		)
 		(property "Value" "PHOENIX_MKDSO_2.5_3_R"
-			(at 284.48 74.9299 0)
+			(at 258.572 66.548 0)
 			(show_name no)
 			(do_not_autoplace no)
@@
 		(in_pos_files yes)
 		(dnp no)
-		(fields_autoplaced yes)
 		(property "Reference" "J6"
-			(at 284.48 96.5199 0)
+			(at 280.67 88.392 0)
 			(show_name no)
 			(do_not_autoplace no)
@@
 		)
 		(property "Value" "PHOENIX_MKDSO_2.5_3_R"
-			(at 284.48 99.0599 0)
+			(at 258.826 90.678 0)
 			(show_name no)
 			(do_not_autoplace no)
